File: europa.kicad_pcb (KiCad board)
At the start: 2 copper layers, 40.3 x 128.5 mm, 17 parts, among them J1 Left, J2 Right, J3 AudioJack2_Ground, J4 AudioJack2_Ground, J5 AudioJack2_Ground, J6 AudioJack2_Ground

Commit message: Layout finished, needs tweak in proper components
Parts:
- R2, R3, R4: value R_Small -> 12k
- RV1, RV2, RV3: value 5K -> 5k
- moved R4 28.7 mm to (113.8, 95.0)
- moved R1 20.7 mm to (99.6, 24.4), turned to 0 degrees
- moved J1 17.8 mm to (111.0, 85.7)
- moved J2 17.8 mm to (93.2, 85.7)
- moved R2 14.2 mm to (84.8, 95.0)
- moved R3 13.7 mm to (99.6, 95.0)
Connections:
- J1 pad 10: /IOB_23B -> VREF
- J1 pad 12: /IOB_29B -> AU_OUT1
- J1 pad 14: /IOB_20A -> BUTTON2
- J1 pad 15: /IOB_16A -> BUTTON1
- J1 pad 18: /IOB_8A -> A1
- J1 pad 19: A0 -> VREF
- J1 pad 20: VREF -> A0
- J1 pad 21: A1 -> VREF
- J1 pad 22: VREF -> /IOB_2A
- J1 pad 23: A2 -> /IOB_0A
- J1 pad 24: VREF -> /IOB_6A
- J1 pad 6: /IOB_18A -> BUTTON3
- J1 pad 9: /IOB_22A -> AU_IN1
- J2 pad 11: /IOT_37A -> A2
- J2 pad 12: /IOT_36B -> VREF
- J2 pad 24: VREF -> /IOT_41A
- J3 pad S: unconnected-(J3-PadS) -> AU_IN1
- J3 pad T: unconnected-(J3-PadT) -> GND
- J4 pad T: unconnected-(J4-PadT) -> GND
- J5 pad S: unconnected-(J5-PadS) -> AU_OUT1
- J5 pad T: unconnected-(J5-PadT) -> GND
- J6 pad T: unconnected-(J6-PadT) -> GND
- OBSTAIN1 pad 1: Net-(R4-Pad1) -> BUTTON3
- PING1 pad 1: Net-(R3-Pad1) -> BUTTON2
- R2 pad 1: Net-(R2-Pad1) -> BUTTON1
- R3 pad 1: Net-(R3-Pad1) -> BUTTON2
- R4 pad 1: Net-(R4-Pad1) -> BUTTON3
- RV1 pad 1: +5VD -> +3V3
- RV2 pad 1: +5VD -> +3V3
- RV3 pad 1: +5VD -> +3V3
- THWART1 pad 1: Net-(R2-Pad1) -> BUTTON1
Routing:
- net AU_OUT1: track 0.00 -> 81.2 mm
- net BUTTON1: track 0.00 -> 73.5 mm
- net VREF: track 0.00 -> 65.8 mm
- net BUTTON2: track 0.00 -> 56.8 mm
- net AU_IN1: track 0.00 -> 56.2 mm
- net +3V3: track 0.00 -> 51.4 mm
- net BUTTON3: track 0.00 -> 33.0 mm
- net A2: track 0.00 -> 21.3 mm
- net A1: track 0.00 -> 21.3 mm
- net A0: track 0.00 -> 10.8 mm
- net REF_CLK: track 0.00 -> 8.59 mm
- added copper zone on F.Cu, net +3V3
- added copper zone on B.Cu, net GND

Commit message: Mono plugs now connecting properly. Switches found at farnell
Parts:
- J3: value AudioJack2_Ground -> AudioJack2
Connections:
- J3 pad S: AU_IN1 -> GND
- J3 pad T: GND -> AU_IN1
- J4 pad S: unconnected-(J4-PadS) -> GND
- J4 pad T: GND -> unconnected-(J4-PadT)
- J5 pad S: AU_OUT1 -> GND
- J5 pad T: GND -> AU_OUT1
- J6 pad S: unconnected-(J6-PadS) -> GND
- J6 pad T: GND -> unconnected-(J6-PadT)
Routing:
- net AU_OUT1: track 81.2 -> 92.6 mm
- net AU_IN1: track 56.2 -> 66.5 mm
Changed lines of the file:
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@@
   (net 41 "AU_IN1")
   (net 42 "AU_OUT1")
-  (net 43 "unconnected-(J4-PadS)")
-  (net 44 "unconnected-(J6-PadS)")
+  (net 43 "unconnected-(J4-PadT)")
+  (net 44 "unconnected-(J6-PadT)")
   (net 45 "/IOT_41A")
   (footprint "josh-buttons-switches:SW_Push_KMR2" (layer "F.Cu")
@@
     (fp_circle (center 0 6.48) (end 1.8 6.48) (layer "F.Fab") (width 0.1) (fill none))
     (pad "S" thru_hole rect (at 0 0 180) (locked) (size 1.93 1.83) (drill 1.22) (layers *.Cu *.Mask)
-      (net 43 "unconnected-(J4-PadS)") (pintype "passive"))
+      (net 14 "GND") (pintype "passive"))
     (pad "T" thru_hole circle (at 0 11.4 180) (locked) (size 2.13 2.13) (drill 1.43) (layers *.Cu *.Mask)
-      (net 14 "GND") (pintype "passive"))
+      (net 43 "unconnected-(J4-PadT)") (pintype "passive"))
     (pad "TN" thru_hole circle (at 0 3.1 180) (locked) (size 2.13 2.13) (drill 1.42) (layers *.Cu *.Mask))
     (model "${KICAD6_3DMODEL_DIR}/Connector_Audio.3dshapes/Jack_3.5mm_QingPu_WQP-PJ398SM_Vertical.wrl"
@@
     (fp_circle (center 0 6.48) (end 1.8 6.48) (layer "F.Fab") (width 0.1) (fill none))
     (pad "S" thru_hole rect (at 0 0 180) (locked) (size 1.93 1.83) (drill 1.22) (layers *.Cu *.Mask)
-      (net 44 "unconnected-(J6-PadS)") (pintype "passive"))
+      (net 14 "GND") (pintype "passive"))
     (pad "T" thru_hole circle (at 0 11.4 180) (locked) (size 2.13 2.13) (drill 1.43) (layers *.Cu *.Mask)
-      (net 14 "GND") (pintype "passive"))
+      (net 44 "unconnected-(J6-PadT)") (pintype "passive"))
     (pad "TN" thru_hole circle (at 0 3.1 180) (locked) (size 2.13 2.13) (drill 1.42) (layers *.Cu *.Mask))
     (model "${KICAD6_3DMODEL_DIR}/Connector_Audio.3dshapes/Jack_3.5mm_QingPu_WQP-PJ398SM_Vertical.wrl"
@@
       (effects (font (size 1 1) (thickness 0.15)))
     )
-    (fp_text value "AudioJack2_Ground" (at 0 5 180) (layer "F.Fab")
+    (fp_text value "AudioJack2" (at 0 5 180) (layer "F.Fab")
       (effects (font (size 1 1) (thickness 0.15)))
     )
@@
     (fp_circle (center 0 6.48) (end 1.8 6.48) (layer "F.Fab") (width 0.1) (fill none))
     (pad "S" thru_hole rect (at 0 0 180) (locked) (size 1.93 1.83) (drill 1.22) (layers *.Cu *.Mask)
+      (net 14 "GND") (pintype "passive"))
+    (pad "T" thru_hole circle (at 0 11.4 180) (locked) (size 2.13 2.13) (drill 1.43) (layers *.Cu *.Mask)
       (net 41 "AU_IN1") (pintype "passive"))
-    (pad "T" thru_hole circle (at 0 11.4 180) (locked) (size 2.13 2.13) (drill 1.43) (layers *.Cu *.Mask)
-      (net 14 "GND") (pintype "passive"))
     (pad "TN" thru_hole circle (at 0 3.1 180) (locked) (size 2.13 2.13) (drill 1.42) (layers *.Cu *.Mask))
     (model "${KICAD6_3DMODEL_DIR}/Connector_Audio.3dshapes/Jack_3.5mm_QingPu_WQP-PJ398SM_Vertical.wrl"
@@
     (fp_circle (center 0 6.48) (end 1.8 6.48) (layer "F.Fab") (width 0.1) (fill none))
     (pad "S" thru_hole rect (at 0 0 180) (locked) (size 1.93 1.83) (drill 1.22) (layers *.Cu *.Mask)
+      (net 14 "GND") (pintype "passive"))
+    (pad "T" thru_hole circle (at 0 11.4 180) (locked) (size 2.13 2.13) (drill 1.43) (layers *.Cu *.Mask)
       (net 42 "AU_OUT1") (pintype "passive"))
-    (pad "T" thru_hole circle (at 0 11.4 180) (locked) (size 2.13 2.13) (drill 1.43) (layers *.Cu *.Mask)
-      (net 14 "GND") (pintype "passive"))
     (pad "TN" thru_hole circle (at 0 3.1 180) (locked) (size 2.13 2.13) (drill 1.42) (layers *.Cu *.Mask))
     (model "${KICAD6_3DMODEL_DIR}/Connector_Audio.3dshapes/Jack_3.5mm_QingPu_WQP-PJ398SM_Vertical.wrl"
@@
   (segment (start 85.072 102.146) (end 89.172 102.146) (width 0.25) (layer "F.Cu") (net 33))
   (segment (start 85.072 102.146) (end 118.382 102.146) (width 0.25) (layer "F.Cu") (net 33))
-  (segment (start 112.175011 92.548989) (end 112.175011 66.525011) (width 0.25) (layer "B.Cu") (net 41))
-  (segment (start 93.344 111.38) (end 112.175011 92.548989) (width 0.25) (layer "B.Cu") (net 41))
-  (segment (start 91.44 111.38) (end 93.344 111.38) (width 0.25) (layer "B.Cu") (net 41))
+  (segment (start 112.175011 93.436565) (end 112.175011 66.525011) (width 0.25) (layer "B.Cu") (net 41))
+  (segment (start 97.028 108.583576) (end 112.175011 93.436565) (width 0.25) (layer "B.Cu") (net 41))
+  (segment (start 97.028 117.192) (end 97.028 108.583576) (width 0.25) (layer "B.Cu") (net 41))
   (segment (start 112.175011 66.525011) (end 111 65.35) (width 0.25) (layer "B.Cu") (net 41))
-  (segment (start 91.44 128.078) (end 99.06 120.458) (width 0.25) (layer "B.Cu") (net 42))
-  (segment (start 99.06 107.188) (end 114.817011 91.430989) (width 0.25) (layer "B.Cu") (net 42))
+  (segment (start 91.44 122.78) (end 97.028 117.192) (width 0.25) (layer "B.Cu") (net 41))
+  (segment (start 98.552 107.696) (end 114.817011 91.430989) (width 0.25) (layer "B.Cu") (net 42))
+  (segment (start 91.44 139.478) (end 98.552 132.366) (width 0.25) (layer "B.Cu") (net 42))
   (segment (start 114.817011 61.547011) (end 111.318212 58.048212) (width 0.25) (layer "B.Cu") (net 42))
   (segment (start 114.817011 91.430989) (end 114.817011 61.547011) (width 0.25) (layer "B.Cu") (net 42))
-  (segment (start 99.06 120.458) (end 99.06 107.188) (width 0.25) (layer "B.Cu") (net 42))
+  (segment (start 98.552 132.366) (end 98.552 107.696) (width 0.25) (layer "B.Cu") (net 42))
   (zone (net 33) (net_name "+3V3") (layer "F.Cu") (hatch edge 0.508)
     (connect_pads (clearance 0.508))
